File: kicad/MOnkShield.sch (KiCad schematic (older format))
At the start: 1 part

Commit message: add CHIP-DIPs library, start connecting the dots
Parts:
- added C1: .1uF, symbol C
- added C2: 10uF, symbol CP
- added J1, J2: DIP-HEADER-2x20, CHIP-DIPs:DIP_Header_2x20, symbol DIP-HEADER-2x20
- added P?: Motor 1, symbol CONN_01X02
- added P?: Motor 2, symbol CONN_01X02
- added P?: VMotor, symbol CONN_01X02
- added P?: PWR_SEL, symbol CONN_01X03
- gave numbers to parts that had none: 1
Connections:
- net labels added: +1.8V, +3.3V, +5V, 3.3+, AP-EINT1, AP-EINT3, CSICK, CSID0, CSID1, CSID2, CSID3, CSID4, CSID5, CSID6, CSID7, CSIHSYNC, CSIPCK, CSIVSYNC, FEL, GND, HPCOM, HPL, HPR, LCD-CLK, LCD-D10, LCD-D11, LCD-D12, LCD-D13, LCD-D14, LCD-D15, LCD-D18, LCD-D19, LCD-D2, LCD-D20, LCD-D21, LCD-D22, LCD-D23, LCD-D3, LCD-D4, LCD-D5, LCD-D6, LCD-D7, LCD-DE, LCD-HSYNC, LCD-VSYNC, LRADC, M1-1, M1-2, M2-1, M2-2, MICIN1, MICM, PWM0, PWRON, TS, TWI1-SCK, TWI1-SDA, TWI2-SCK, TWI2-SDA, UART1-RX, UART1-TX, VBAT, VCHG, VM+, X1, X2, XIO-P0, XIO-P1, XIO-P2, XIO-P3, XIO-P4, XIO-P5, XIO-P6, XIO-P7, Y1, Y2
- wire segments 0 -> 144
Other:
- note added: "CHIP Headers"
- moved on the sheet: U1
